File: pcb/esp.ra.dio/esp.ra.dio.kicad_pcb (KiCad board)
At the start: 2 copper layers, 75 x 28 mm, 33 parts, among them J1 A, J10 UART, J2 B, J3 C, J4 D, J5 START, J6 SELECT, J7 JOY, J8 USB_B_Micro, J9 BATTERY, Q1 BSS138, SW1 POWER, SW2 RESET, SW3 BOOT, U2 VCC, U3 RT9080-33GJ5

Commit message: checkpoint moving to shift reg
Parts:
- added C6: 0.1uF, Capacitor_SMD:C_0805_2012Metric_Pad1.18x1.45mm_HandSolder, F.Cu at (66.8, 85.0)
- added R1: 2M, Resistor_SMD:R_0805_2012Metric_Pad1.20x1.40mm_HandSolder, F.Cu at (51.7, 85.2)
- added R11: 10K, Resistor_SMD:R_0805_2012Metric_Pad1.20x1.40mm_HandSolder, F.Cu at (55.6, 92.9)
- added R12: 10K, Resistor_SMD:R_0805_2012Metric_Pad1.20x1.40mm_HandSolder, F.Cu at (57.3, 99.7)
- added R13: 10K, Resistor_SMD:R_0805_2012Metric_Pad1.20x1.40mm_HandSolder, F.Cu at (62.0, 85.0)
- added R14: 10K, Resistor_SMD:R_0805_2012Metric_Pad1.20x1.40mm_HandSolder, F.Cu at (62.0, 87.9)
- added R15: 10K, Resistor_SMD:R_0805_2012Metric_Pad1.20x1.40mm_HandSolder, F.Cu at (62.0, 90.9)
- added R16: 10K, Resistor_SMD:R_0805_2012Metric_Pad1.20x1.40mm_HandSolder, F.Cu at (62.0, 93.8)
- added R2: 2M, Resistor_SMD:R_0805_2012Metric_Pad1.20x1.40mm_HandSolder, F.Cu at (47.1, 87.5)
- added R5: 10K, Resistor_SMD:R_0805_2012Metric_Pad1.20x1.40mm_HandSolder, F.Cu at (61.0, 81.5)
- added R6: 10K, Resistor_SMD:R_0805_2012Metric_Pad1.20x1.40mm_HandSolder, F.Cu at (57.7, 86.9)
- added U4: SN74LV165APWRG3, SN74LV:SOP65P640X120-16N, F.Cu at (101.1, 53.0)
- Q1: value BSS138 -> BSS84
- R10: value 1M -> 10K
- R4: value 4.7K -> 10K
- R7: value 1M -> 100K
Connections:
- D1 pad 2: VCC -> /ACTLED
- Q1 pad 1: /ACTLED -> /~{VCC_SW_EN}
- Q1 pad 2: GND -> VCC
- Q1 pad 3: Net-(Q1-D) -> VCC_SW
- R10 pad 1: /ACTLED -> VCC_SW
- R10 pad 2: GND -> /BC
- R4 pad 2: Net-(Q1-D) -> GND
- R7 pad 2: /ACTLED -> /~{VCC_SW_EN}
- R8 pad 1: /BA -> Net-(U2-GPIO20/U0RXD)
- R9 pad 1: /BD -> Net-(U2-GPIO21/U0TXD)
- U2 pad 10: /BC -> /~{VCC_SW_EN}
- U2 pad 11: /BA -> Net-(U2-GPIO20/U0RXD)
- U2 pad 12: /BD -> Net-(U2-GPIO21/U0TXD)
- U2 pad 15: /BB -> /ACTLED
- U2 pad 16: /GPIO2 -> /BATSENSE
- U2 pad 3: /DL -> /SCLK
- U2 pad 4: /DR -> /MISO
- U2 pad 5: /DD -> unconnected-(U2-GPIO6-Pad5)
- U2 pad 6: /DU -> /~{LATCH}
- U2 pad 7: /ACTLED -> Net-(U2-GPIO8)
Routing:
- net /GPIO2: track 26.8 -> 0.00 mm, vias 2 -> 0
- net /BATSENSE: track 0.00 -> 26.8 mm, vias 0 -> 2
- net Net-(Q1-D): track 3.50 -> 0.00 mm
- net GND: track 6.34 -> 9.83 mm, vias 17 -> 16
- net /BC: vias 0 -> 1

Commit message: Routing checkpoint
Parts:
- JP1: value USB Power -> Sense Ground; footprint Jumper:SolderJumper-2_P1.3mm_Open_TrianglePad1.0x1.5mm -> Jumper:SolderJumper-3_P1.3mm_Open_Pad1.0x1.5mm_NumberLabels
- R1, R2: value 2M -> 1M
- R7: value 100K -> 10K
- moved JP1 62.5 mm to (110.0, 69.8), turned to 0 degrees
- moved R11 46.3 mm to (96.0, 70.2), turned to 90 degrees
- moved J10 45.6 mm to (46.2, 75.5), turned to 90 degrees
- moved Q1 39.6 mm to (47.9, 66.2), turned to -90 degrees
- moved R12 38.8 mm to (86.8, 74.5), turned to 90 degrees
- moved R15 37.7 mm to (96.0, 74.5), turned to 90 degrees
- moved R6 36.2 mm to (89.8, 70.2), turned to 90 degrees
- moved R2 34.2 mm to (78.8, 74.5), turned to -90 degrees
- moved R14 33.7 mm to (92.9, 74.5), turned to 90 degrees
- moved R9 31.6 mm to (48.0, 69.8), turned to 180 degrees
- moved R1 31.2 mm to (81.0, 74.5), turned to -90 degrees
- moved R7 30.2 mm to (51.8, 66.2), turned to -90 degrees
- moved R13 29.7 mm to (89.8, 74.5), turned to 90 degrees
- moved R16 28.7 mm to (54.2, 66.2), turned to 90 degrees
- moved R5 28.1 mm to (86.8, 70.2), turned to 90 degrees
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Connections:
- C4 pad 1: Net-(JP1-B) -> /VBUS
- JP1 pad 1: /VBUS -> GND
- JP1 pad 2: Net-(JP1-B) -> Net-(JP1-C)
- R2 pad 1: GND -> Net-(JP1-C)
- SW1 pad 2: Net-(JP1-B) -> /VBUS
- U2 pad 5: unconnected-(U2-GPIO6-Pad5) -> /BATSENSE_SINK
- U3 pad 1: Net-(JP1-B) -> /VBUS
- U3 pad 3: Net-(JP1-B) -> /VBUS
Routing:
- net VCC: track 108.3 -> 40.6 mm, vias 1 -> 0
- net /ACTLED: track 36.5 -> 0.00 mm, vias 2 -> 0
- net /USB_DP: track 33.4 -> 0.00 mm, vias 2 -> 0
- net /USB_DN: track 33.4 -> 0.00 mm, vias 2 -> 0
- net /BD: track 48.8 -> 17.5 mm, vias 0 -> 1
- net /STA: track 27.0 -> 0.00 mm
- net /BATSENSE: track 26.8 -> 0.00 mm, vias 2 -> 0
- net Net-(JP1-B): track 25.4 -> 0.00 mm
- net /SEL: track 18.3 -> 0.10 mm
- net /BB: track 25.7 -> 7.56 mm, vias 0 -> 1
- net /BA: track 48.5 -> 33.1 mm, vias 0 -> 1
- net /DL: track 23.5 -> 34.7 mm, vias 1 -> 2
- net /TX: track 10.9 -> 0.00 mm
- net /BC: track 27.7 -> 18.0 mm
- net /RX: track 8.93 -> 0.00 mm
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
Commit message: Horrible routing job done
Parts:
- removed R10, R11, R12, R13, R14, R15, R5, R6: 10K, Resistor_SMD:R_0805_2012Metric_Pad1.20x1.40mm_HandSolder
- added RN1: R_Network08_US, RN:RN, F.Cu at (96.8, 71.8)
- moved C6 26.1 mm to (109.0, 70.1)
- moved R1 26.1 mm to (106.8, 70.1), turned to 90 degrees
- moved R2 26.1 mm to (104.5, 70.1)
- moved U4 12.3 mm to (89.8, 71.8)
- moved JP1 9.95 mm to (102.1, 75.8)
- moved R3 2.10 mm to (60.6, 74.5)
- moved C3 1.30 mm to (62.8, 74.5)
Routing:
- net /VBAT: track 11.1 -> 100.5 mm, vias 0 -> 1
- net VCC_SW: track 0.00 -> 59.2 mm, vias 0 -> 3
- net /BATSENSE_SINK: track 0.00 -> 52.8 mm, vias 0 -> 2
- net /MISO: track 0.00 -> 45.0 mm, vias 0 -> 2
- net /BATSENSE: track 0.00 -> 40.5 mm, vias 0 -> 2
- net /USB_DP: track 0.00 -> 38.1 mm, vias 0 -> 2
- net /SCLK: track 0.00 -> 37.3 mm
- net /USB_DN: track 0.00 -> 36.8 mm, vias 0 -> 2
- net Net-(U2-GPIO20/U0RXD): track 0.00 -> 34.2 mm, vias 0 -> 2
- net /~{LATCH}: track 0.00 -> 33.8 mm
- net Net-(U2-GPIO21/U0TXD): track 0.00 -> 32.9 mm, vias 0 -> 2
- net /STA: track 0.00 -> 26.5 mm, vias 0 -> 1
- net /~{VCC_SW_EN}: track 3.72 -> 28.0 mm, vias 0 -> 2
- net /BB: track 7.56 -> 28.6 mm
- net /SEL: track 0.10 -> 19.5 mm, vias 0 -> 1
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