File: pcb/esp.ra.dio/esp.ra.dio.kicad_sch (KiCad schematic)
At the start: 45 parts, among them J1 A, J10 UART, J2 B, J3 C, J4 D, J5 START, J6 SELECT, J7 JOY, J8 USB_B_Micro, J9 BATTERY, Q1 BSS84, SW1 POWER, SW2 RESET, SW3 BOOT, U2 VCC, U3 RT9080-33GJ5, U4 SN74LV165APWRG3

Commit message: checkpoint moving to shift reg
Parts:
- R4: value 4.7K -> 10K
- U4: footprint SN74LV165APWRG3:SOP65P640X120-16N -> SN74LV:SOP65P640X120-16N
Changed lines of the file:
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@@
 		)
 	)
-	(text_box "GPIO8 strapping pin\nDEV: always 1 for either boot condition.\nPROD: always 0, unable to joint boot\nPost boot, drive low current LED\nIf we left the pullup in permanently, would leak"
-		(exclude_from_sim no)
-		(at 236.22 121.92 0)
-		(size 43.18 14.1714)
-		(margins 0.9525 0.9525 0.9525 0.9525)
-		(stroke
-			(width 0)
-			(type solid)
-		)
-		(fill
-			(type none)
-		)
-		(effects
-			(font
-				(size 1.27 1.27)
-			)
-			(justify left top)
-		)
-	)
 	(text_box "// ESP32-C3 DEFAULT PINS\nstatic const uint8_t SDA = 8;\nstatic const uint8_t SCL = 9;\nstatic const uint8_t SS = 7;\nstatic const uint8_t MOSI = 6;\nstatic const uint8_t MISO = 5;\nstatic const uint8_t SCK = 4;\n\n"
 		(exclude_from_sim no)
@@
 			)
 		)
-		(property "Footprint" "SN74LV165APWRG3:SOP65P640X120-16N"
+		(property "Footprint" "SN74LV:SOP65P640X120-16N"
 			(at 87.63 134.62 0)
 			(hide yes)
@@
 			)
 		)
-		(property "Value" "4.7K"
+		(property "Value" "10K"
 			(at 210.82 106.68 90)
 			(show_name no)

Commit message: Schematic
Parts:
- removed JP1: USB Power, Jumper:SolderJumper-2_P1.3mm_Open_TrianglePad1.0x1.5mm, symbol Jumper:Jumper_2_Open
- added JP1: Sense Ground, Jumper:SolderJumper-3_P1.3mm_Open_Pad1.0x1.5mm_NumberLabels, symbol Jumper:SolderJumper_3_Open
- R1, R2: value 2M -> 1M
- R7: value 100K -> 10K
Connections:
- net GND: now also JP1.1 (A); no longer R2.1
- net VBUS: now also C4.1, SW1.2 (B), U3.1 (IN), U3.3 (EN)
- net BATSENSE_SINK: now reaches U2.5 (GPIO6)
- net BATSENSE_SINK: now also JP1.3 (B)
- new net: JP1.2 (C), R2.1
- no-connect marks 4 -> 3
Other:
- moved on the sheet: R2, R8, R9

Commit message: Horrible routing job done
Parts:
- removed R10, R11, R12, R13, R14, R15, R5, R6: 10K, Resistor_SMD:R_0805_2012Metric_Pad1.20x1.40mm_HandSolder, symbol Device:R_Small
- added RN1: 10K, RN:RN, symbol Device:R_Network08_US
Connections:
- net BA: now also RN1.9 (R8)
- net BB: now also RN1.8 (R7)
- net BC: now also RN1.7 (R6)
- net BD: now also RN1.6 (R5)
- net DD: now also RN1.4 (R3)
- net DL: now also RN1.2 (R1)
- net DR: now also RN1.3 (R2)
- net DU: now also RN1.5 (R4)
- net VCC_SW: now also RN1.1 (common)
